File: power_glitcher/power_glitcher.kicad_pcb (KiCad board)
At the start: 2 copper layers, 46.3 x 40.2 mm, 60 parts, among them J1 Conn_01x09, J2 Conn_01x02, J3 Conn_01x02, J4 Conn_01x02, J5 Conn_01x02, Q1 BC817, Q2 BC807, U1 AD9708AR, U2 Opamp_Dual, U3 TL081H, U5 LM2735XMF

Commit message: Rev 2.0
Parts:
- removed JP2: SolderJumper_2_Open, Jumper:SolderJumper-2_P1.3mm_Open_Pad1.0x1.5mm
- added C21: 0.1uF, Capacitor_SMD:C_0805_2012Metric, F.Cu at (102.9, 87.9)
- added C22: 1uF, Capacitor_SMD:C_0805_2012Metric, F.Cu at (102.9, 90.1)
- added C23: 10uF, Capacitor_SMD:C_0805_2012Metric, F.Cu at (111.3, 67.1)
- added C24: 10uF, Capacitor_SMD:C_0805_2012Metric, F.Cu at (121.8, 65.8)
- added C25: 0.1uF, Capacitor_SMD:C_0805_2012Metric, F.Cu at (94.6, 91.4)
- added J6: Conn_01x02, Connector_PinHeader_2.54mm:PinHeader_1x02_P2.54mm_Vertical, F.Cu at (112.4, 75.8)
- added U4: ICL7660, Package_SO:SO-8_3.9x4.9mm_P1.27mm, F.Cu at (116.6, 67.4)
- moved L1 7.38 mm to (106.7, 66.6)
- moved J5 3.35 mm to (108.7, 71.1), turned to -90 degrees
- moved U3 1.38 mm to (94.6, 88.2)
- moved D1 1.27 mm to (118.6, 81.9)
- moved J4 1.27 mm to (123.9, 72.1)
- moved Q1 1.27 mm to (123.0, 80.2)
- moved Q2 1.27 mm to (122.9, 90.6)
- moved R18 1.27 mm to (118.4, 87.1)
- moved R19 1.27 mm to (118.5, 84.4)
- moved R2 1.27 mm to (122.8, 86.8)
- moved R3 1.27 mm to (122.9, 75.7)
- moved C1 1.27 mm to (118.1, 71.8)
- moved D2 1.27 mm to (118.4, 89.4)
- moved R1 1.27 mm to (122.7, 84.6)
- moved R11 1.27 mm to (118.2, 74.0)
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Connections:
- C11 pad 1: AVCC -> V+
- C12 pad 1: AVCC -> V-
- C13 pad 1: AVCC -> V+
- U2 pad 4: AGND -> V-
- U2 pad 8: AVCC -> V+
- U3 pad 2: AVCC -> V-
- U3 pad 5: AGND -> V+
Routing:
- net V-: track 11.9 -> 79.8 mm, vias 0 -> 2
- net V+: track 31.7 -> 80.9 mm, vias 0 -> 3
- net AVCC: track 125.2 -> 106.4 mm, vias 0 -> 2
- net Net-(R1-Pad2): track 48.0 -> 38.1 mm
- net Net-(R16-Pad1): track 23.9 -> 29.2 mm
- net Net-(D3-A): track 10.5 -> 14.7 mm
- net Net-(U4-CAP-): track 0.00 -> 3.24 mm
- net Net-(U4-CAP+): track 0.00 -> 2.97 mm
- net Net-(U3--): track 5.95 -> 8.13 mm
- net Net-(J5-Pin_1): track 8.81 -> 6.97 mm
- net /reflo: track 11.4 -> 12.6 mm
- net AGND: track 190.0 -> 188.8 mm
Other:
- board text added: "Power Glitcher rev2.0"
- board text added: "V+"
- board text added: "V-"
- board text removed: "Power Glitcher v1.0"

Commit message: Add bypass jumper for LM2735 and power analysis capability
Parts:
- added J7: Conn_01x02, Connector_PinHeader_2.54mm:PinHeader_1x02_P2.54mm_Vertical, F.Cu at (124.3, 65.9)
- added JP2: SolderJumper_2_Open, Jumper:SolderJumper-2_P1.3mm_Open_Pad1.0x1.5mm, F.Cu at (102.6, 69.7)
- added R23: 1, Resistor_SMD:R_0805_2012Metric, F.Cu at (121.0, 65.7)
- C1: value C -> 1pF
- R10: value R -> 100
- R11: value R -> 4K7
- R18, R19: value R -> 0
- R7: value R -> 64.9
- moved C24 3.73 mm to (121.0, 69.5)
- moved U4 1.56 mm to (115.1, 67.4)
- moved L1 1.41 mm to (105.4, 66.0)
- moved C23 1.40 mm to (109.9, 67.0)
- moved J4 0.74 mm to (124.3, 72.7)
- moved R3 0.33 mm to (122.9, 76.1)
- moved C16 0.13 mm to (97.3, 74.1)
- moved C17 0.13 mm to (99.6, 74.1)
Connections:
- J4 pad 2: AGND -> Net-(J4-Pin_2)
Routing:
- net V+: track 80.9 -> 91.5 mm
- net Net-(J4-Pin_2): track 0.00 -> 7.76 mm
- net AGND: track 188.8 -> 184.9 mm, vias 12 -> 13
- net AVCC: track 106.4 -> 104.2 mm
- net V-: track 79.8 -> 78.3 mm
- net Net-(R1-Pad2): track 38.1 -> 37.2 mm
- net Net-(U4-CAP-): track 3.24 -> 2.47 mm
Other:
- board text added: "Power Glitcher rev3.0"
- board text removed: "Power Glitcher rev2.0"
- board text removed: "Vout"
