File: power_glitcher/power_glitcher.kicad_sch (KiCad schematic)
At the start: 60 parts, among them J1 Conn_01x09, J2 Conn_01x02, J3 Conn_01x02, J4 Conn_01x02, J5 Conn_01x02, Q1 BC817, Q2 BC807, U1 AD9708AR, U2 Opamp_Dual, U3 TL081H, U5 LM2735XMF

Commit message: Rev 2.0
Parts:
- removed JP2: SolderJumper_2_Open, Jumper:SolderJumper-2_P1.3mm_Open_Pad1.0x1.5mm, symbol Jumper:SolderJumper_2_Open
- added C21, C25: 0.1uF, Capacitor_SMD:C_0805_2012Metric, symbol Device:C
- added C22: 1uF, Capacitor_SMD:C_0805_2012Metric, symbol Device:C
- added C23, C24: 10uF, Capacitor_SMD:C_0805_2012Metric, symbol Device:C
- added J6: Conn_01x02, Connector_PinHeader_2.54mm:PinHeader_1x02_P2.54mm_Vertical, symbol Connector_Generic:Conn_01x02
- added U4: ICL7660, Package_SO:SO-8_3.9x4.9mm_P1.27mm, symbol Regulator_SwitchedCapacitor:ICL7660
Connections:
- net AGND: now also C21.2, C22.2, C24.2, C25.1, U4.3 (GND); no longer U2.4 (V-), U3.5 (V+)
- net AVCC: no longer C11.1, C12.1, C13.1, U2.8 (V+), U3.2 (V-)
- net V+: now also C11.1, C13.1, U2.8 (V+), U3.5 (V+), C25.2, J6.1 (Pin_1), U4.8 (V+)
- net V-: now also C12.1, U2.4 (V-), U3.2 (V-), C21.1, C22.1, C24.1, J6.2 (Pin_2), U4.5 (VOUT)
- new net: C23.1, U4.2 (CAP+)
- new net: C23.2, U4.4 (CAP-)
Other:
- moved on the sheet: J5, JP1, U2C

Commit message: Update BOM
Parts:
- C1: value C -> 1pF
- R10: value R -> 100
- R11: value R -> 4K7
- R18, R19: value R -> 0
- R7: value R -> 64.9
Changed lines of the file:
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@@
 	(title_block
 		(title "Power Glitcher")
-		(date "2024-11-17")
-		(rev "2.0")
+		(date "2024-11-24")
+		(rev "2.1")
 		(company "Carles Pey")
 	)
@@
 			)
 		)
-		(property "Value" "R"
+		(property "Value" "0"
 			(at 213.614 97.536 0)
 			(effects
@@
 			)
 		)
-		(property "Value" "R"
+		(property "Value" "0"
 			(at 213.36 87.376 0)
 			(effects
@@
 			)
 		)
-		(property "Value" "R"
+		(property "Value" "64.9"
 			(at 182.88 91.44 90)
 			(effects
@@
 			)
 		)
-		(property "Value" "R"
+		(property "Value" "100"
 			(at 135.89 105.4099 0)
 			(effects
@@
 			)
 		)
-		(property "Value" "C"
+		(property "Value" "1pF"
 			(at 247.65 106.6799 0)
 			(effects
@@
 			)
 		)
-		(property "Value" "R"
+		(property "Value" "4K7"
 			(at 246.38 99.0599 0)
 			(effects

Commit message: Add bypass jumper for LM2735 and power analysis capability
Parts:
- added J7: Conn_01x02, Connector_PinHeader_2.54mm:PinHeader_1x02_P2.54mm_Vertical, symbol Connector_Generic:Conn_01x02
- added JP2: SolderJumper_2_Open, Jumper:SolderJumper-2_P1.3mm_Open_Pad1.0x1.5mm, symbol Jumper:SolderJumper_2_Open
- added R23: 1, Resistor_SMD:R_0805_2012Metric, symbol Device:R_US
Connections:
- net AGND: now also J7.2 (Pin_2), R23.1; no longer J4.2 (Pin_2)
- net AVCC: now also JP2.2 (B)
- net V+: now also JP2.1 (A)
- new net: J4.2 (Pin_2), J7.1 (Pin_1), R23.2
Other:
- note added: "SCA"
- moved on the sheet: C3
